Commit message: changed body link to base_footprint to match with standards

File: urdf/neato.urdf (robot description, URDF)
Before this commit: robot neato, 5 links, 4 joints
Links:
- removed link body
- added link base_footprint; visual box size=0.33 0.165 0.074; visual cylinder length=0.074 radius=0.165
Joints:
- removed joint body_joint
- added joint base_footprint_joint: type fixed, parent base_link, child base_footprint, origin xyz=0 0 0.037 rpy=0 0 0

File: urdf/neato.urdf.xacro (robot description, xacro)
@@ -27,5 +27,5 @@
    </material>
    <link name="base_link" />
-   <link name="body">
+   <link name="base_footprint">
       <visual>
          <!--actual: <origin xyz="0 .060 0" rpy="0 0 0" /> -->
@@ -44,7 +44,7 @@
       </visual>
    </link>
-   <joint name="body_joint" type="fixed">
-      <origin xyz="0 0 ${bodyHeight/2}" rpy="0 0 ${pi/2}" />
-      <child link="body" />
+   <joint name="base_footprint_joint" type="fixed">
+      <origin xyz="0 0 ${bodyHeight/2}" rpy="0 0 0" />
+      <child link="base_footprint" />
       <parent link="base_link" />
    </joint>

Commit message: made base_footprint link right above base_link without rotation and fixed bugs regarding the visual when changing rpy for base_link -> base_footprint joint

File: urdf/neato.urdf (robot description, URDF)
Before this commit: robot neato, 5 links, 4 joints
Joints:
- removed joint base_footprint_joint
- added joint body_joint: type fixed, parent base_link, child base_footprint, origin xyz=0 0 0.037 rpy=0 0 0

File: urdf/neato.urdf.xacro (robot description, xacro)
@@ -1,94 +1,94 @@
-<?xml version="1.0" encoding="UTF-8"?>
+<?xml version="1.0"?>
 <robot xmlns:xacro="http://ros.org/wiki/xacro" name="neato">
-   <!-- bodyRadius: half of body width -->
-   <!-- bodyHeight: body height from base to top, excluding casters and wheels -->
-   <!-- laserRadius: radius of outermost laser body -->
-   <!-- laserHeight: distance from of top of body to top of laser body -->
-   <!-- laserRearOffset: distance from rear of body to rear of laser -->
-   <!-- groundClearance: body to ground at rest -->
-   <!-- wheelTrack: distance between wheel centerline -->
-   <!-- wheelZOffset: distance from bottom of body to center of wheel at rest -->
-   <xacro:property name="bodyRadius" value="0.165" />
-   <xacro:property name="bodyRadius2" value="0.0825" />
-   <xacro:property name="bodyHeight" value="0.074" />
-   <xacro:property name="laserRadius" value="0.048" />
-   <xacro:property name="laserHeight" value="0.016" />
-   <xacro:property name="laserRearOffset" value="0.024" />
-   <xacro:property name="groundClearance" value="0.0095" />
-   <xacro:property name="wheelRadius" value="${0.075/2}" />
-   <xacro:property name="wheelWidth" value="0.015" />
-   <xacro:property name="wheelTrack" value="0.238" />
-   <xacro:property name="wheelZOffset" value="${wheelRadius-groundClearance}" />
-   <material name="black">
-      <color rgba="0 0 0 1" />
-   </material>
-   <material name="grey">
-      <color rgba=".5 .5 .5 1" />
-   </material>
-   <link name="base_link" />
-   <link name="base_footprint">
-      <visual>
-         <!--actual: <origin xyz="0 .060 0" rpy="0 0 0" /> -->
-         <origin xyz="0 ${-bodyRadius/2} 0" rpy="0 0 0" />
-         <geometry>
-            <!--actual: <box size="0.330 0.135 0.074"/> -->
-            <box size="${bodyRadius*2} ${bodyRadius} ${bodyHeight}" />
-         </geometry>
-         <material name="black" />
-      </visual>
-      <visual>
-         <geometry>
-            <cylinder length="${bodyHeight}" radius="${bodyRadius}" />
-         </geometry>
-         <material name="black" />
-      </visual>
-   </link>
-   <joint name="base_footprint_joint" type="fixed">
-      <origin xyz="0 0 ${bodyHeight/2}" rpy="0 0 0" />
-      <child link="base_footprint" />
-      <parent link="base_link" />
-   </joint>
-   <link name="sensor_laser">
-      <visual>
-         <geometry>
-            <cylinder radius="${laserRadius}" length="${laserHeight}" />
-         </geometry>
-         <material name="grey" />
-      </visual>
-      <collision>
-         <geometry>
-            <cylinder radius="${laserRadius}" length="${laserHeight}" />
-         </geometry>
-      </collision>
-   </link>
-   <joint name="sensor_laser_joint" type="fixed">
-      <origin xyz="${-(bodyRadius - laserRearOffset - laserRadius)} 0 ${(laserHeight/2) + bodyHeight}" rpy="0 0 0" />
-      <parent link="base_link" />
-      <child link="sensor_laser" />
-   </joint>
-   <xacro:macro name="wheel" params="prefix reflect">
-      <link name="wheel_${prefix}">
-         <visual>
-            <origin xyz="0 0 0" rpy="${pi/2} 0 0" />
+    <!-- bodyRadius: half of body width -->
+    <!-- bodyHeight: body height from base to top, excluding casters and wheels -->
+    <!-- laserRadius: radius of outermost laser body -->
+    <!-- laserHeight: distance from of top of body to top of laser body -->
+    <!-- laserRearOffset: distance from rear of body to rear of laser -->
+    <!-- groundClearance: body to ground at rest -->
+    <!-- wheelTrack: distance between wheel centerline -->
+    <!-- wheelZOffset: distance from bottom of body to center of wheel at rest -->
+    <xacro:property name="bodyRadius" value="0.165" />
+    <xacro:property name="bodyHeight" value="0.074" />
+    <xacro:property name="laserRadius" value="0.048" />
+    <xacro:property name="laserHeight" value="0.016" />
+    <xacro:property name="laserRearOffset" value="0.024" />
+    <xacro:property name="groundClearance" value="0.0095" />
+    <xacro:property name="wheelRadius" value="${0.075/2}" />
+    <xacro:property name="wheelWidth" value="0.015" />
+    <xacro:property name="wheelTrack" value="0.238" />
+    <xacro:property name="wheelZOffset" value="${wheelRadius-groundClearance}" />
+    <material name="black">
+        <color rgba="0 0 0 1" />
+    </material>
+    <material name="grey">
+        <color rgba=".5 .5 .5 1" />
+    </material>
+    <link name="base_link"></link>
+    <link name="base_footprint">
+        <visual>
+            <!--actual: <origin xyz="0 .060 0" rpy="0 0 0" /> -->
+            <origin xyz="${bodyRadius/2} 0 0" rpy="0 0 -1.5708" />
             <geometry>
-               <cylinder length="${wheelWidth}" radius="${wheelRadius}" />
+                <!--actual: <box size="0.330 0.135 0.074"/> -->
+                <box size="${bodyRadius*2} ${bodyRadius} ${bodyHeight}" />
+            </geometry>
+            <material name="black" />
+        </visual>
+        <visual>
+            <geometry>
+                <cylinder length="${bodyHeight}" radius="${bodyRadius}" />
+            </geometry>
+            <material name="black" />
+            <!-- origin xyz="0 0 0" rpy="0 0 1.5708" /-->
+        </visual>
+    </link>
+    <joint name="body_joint" type="fixed">
+        <origin xyz="0 0 ${bodyHeight/2}" rpy="0 0 0" />
+        <child link="base_footprint" />
+        <parent link="base_link" />
+    </joint>
+    <link name="sensor_laser">
+        <visual>
+            <geometry>
+                <cylinder radius="${laserRadius}" length="${laserHeight}" />
             </geometry>
             <material name="grey" />
-         </visual>
-         <collision>
-            <origin xyz="0 0 0" rpy="${pi/2} 0 0" />
+        </visual>
+        <collision>
             <geometry>
-               <cylinder length="${wheelWidth}" radius="${wheelRadius}" />
+                <cylinder radius="${laserRadius}" length="${laserHeight}" />
             </geometry>
-         </collision>
-      </link>
-      <joint name="wheel_${prefix}_joint" type="fixed">
-         <axis xyz="0 1 0" rpy="0 0 0" />
-         <parent link="base_link" />
-         <child link="wheel_${prefix}" />
-         <origin xyz="0 ${reflect * wheelTrack/2} ${wheelZOffset}" rpy="0 0 0" />
-      </joint>
-   </xacro:macro>
-   <xacro:wheel prefix="left" reflect="-1" />
-   <xacro:wheel prefix="right" reflect="1" />
+        </collision>
+    </link>
+    <joint name="sensor_laser_joint" type="fixed">
+        <origin xyz="${-(bodyRadius - laserRearOffset - laserRadius)} 0 ${(laserHeight/2) + bodyHeight}" rpy="0 0 0" />
+        <parent link="base_link" />
+        <child link="sensor_laser" />
+    </joint>
+    <xacro:macro name="wheel" params="prefix reflect">
+        <link name="wheel_${prefix}">
+            <visual>
+                <origin xyz="0 0 0" rpy="${pi/2} 0 0" />
+                <geometry>
+                    <cylinder length="${wheelWidth}" radius="${wheelRadius}" />
+                </geometry>
+                <material name="grey" />
+            </visual>
+            <collision>
+                <origin xyz="0 0 0" rpy="${pi/2} 0 0" />
+                <geometry>
+                    <cylinder length="${wheelWidth}" radius="${wheelRadius}" />
+                </geometry>
+            </collision>
+        </link>
+        <joint name="wheel_${prefix}_joint" type="fixed">
+            <axis xyz="0 1 0" rpy="0 0 0" />
+            <parent link="base_link" />
+            <child link="wheel_${prefix}" />
+            <origin xyz="0 ${reflect * wheelTrack/2} ${wheelZOffset}" rpy="0 0 0" />
+        </joint>
+    </xacro:macro>
+    <xacro:wheel prefix="left" reflect="-1" />
+    <xacro:wheel prefix="right" reflect="1" />
 </robot>

Commit message: Made wheels continuous as to publish live wheel joint position

File: urdf/neato.urdf (robot description, URDF)
Before this commit: robot neato, 5 links, 4 joints
Joints:
- joint wheel_left_joint: type fixed -> continuous
- joint wheel_right_joint: type fixed -> continuous

File: urdf/neato.urdf.xacro (robot description, xacro)
@@ -83,5 +83,5 @@
             </collision>
         </link>
-        <joint name="wheel_${prefix}_joint" type="fixed">
+        <joint name="wheel_${prefix}_joint" type="continuous">
             <axis xyz="0 1 0" rpy="0 0 0" />
             <parent link="base_link" />
